Commit message: Gazebo plugin, collision shapes, launch files, bridge

File: mentorpi_description/urdf/mecanum.xacro (robot description, xacro)
@@ -33,8 +33,6 @@
     </visual>
     <collision>
-      <origin rpy="0 0 0" xyz="0 0 0"/>
-      <geometry>
-        <mesh filename="package://mentorpi_description/meshes/mecanum/base_link.STL"/>
-      </geometry>
+      <origin rpy="0 0 0" xyz="0.0029 0 0.0113"/>
+      <geometry><box size="0.2119 0.1 0.0924"/></geometry>
     </collision>
   </link>
@@ -54,9 +52,7 @@
       </material>
     </visual>
-    <collision>
-      <origin rpy="0 0 0" xyz="0 0 0"/>
-      <geometry>
-        <mesh filename="package://mentorpi_description/meshes/mecanum/wheel_lf_Link.STL"/>
-      </geometry>
+      <collision>
+      <origin rpy="1.5708 0 0" xyz="0 -0.0074 0"/>
+      <geometry><cylinder radius="0.0325" length="0.0344"/></geometry>
     </collision>
   </link>
@@ -82,9 +78,7 @@
       </material>
     </visual>
-    <collision>
-      <origin rpy="0 0 0" xyz="0 0 0"/>
-      <geometry>
-        <mesh filename="package://mentorpi_description/meshes/mecanum/wheel_rf_Link.STL"/>
-      </geometry>
+        <collision>
+      <origin rpy="1.5708 0 0" xyz="0 0.0074 0"/>
+      <geometry><cylinder radius="0.0325" length="0.0344"/></geometry>
     </collision>
   </link>
@@ -110,9 +104,7 @@
       </material>
     </visual>
-    <collision>
-      <origin rpy="0 0 0" xyz="0 0 0"/>
-      <geometry>
-        <mesh filename="package://mentorpi_description/meshes/mecanum/wheel_lb_Link.STL"/>
-      </geometry>
+        <collision>
+      <origin rpy="1.5708 0 0" xyz="0 -0.0074 0"/>
+      <geometry><cylinder radius="0.0325" length="0.0344"/></geometry>
     </collision>
   </link>
@@ -138,9 +130,7 @@
       </material>
     </visual>
-    <collision>
-      <origin rpy="0 0 0" xyz="0 0 0"/>
-      <geometry>
-        <mesh filename="package://mentorpi_description/meshes/mecanum/wheel_rb_Link.STL"/>
-      </geometry>
+        <collision>
+      <origin rpy="1.5708 0 0" xyz="0 0.0074 0"/>
+      <geometry><cylinder radius="0.0325" length="0.0344"/></geometry>
     </collision>
   </link>
@@ -166,10 +156,4 @@
       </material>
     </visual>
-    <collision>
-      <origin rpy="0 0 0" xyz="0 0 0"/>
-      <geometry>
-        <mesh filename="package://mentorpi_description/meshes/mecanum/cam_Link.STL"/>
-      </geometry>
-    </collision>
   </link>
   <joint name="cam_Joint" type="fixed">
@@ -194,10 +178,4 @@
       </material>
     </visual>
-    <collision>
-      <origin rpy="0 0 0" xyz="0 0 0"/>
-      <geometry>
-        <mesh filename="package://mentorpi_description/meshes/mecanum/lidar_Link.STL"/>
-      </geometry>
-    </collision>
   </link>
   <joint name="lidar_Joint" type="fixed">
